File: pcb/datum.kicad_sch (KiCad schematic)
At the start: 46 parts

Commit message: init: rename Sweep Half Swept base to datum
Parts:
- J1, J2: symbol half-swept-rescue:AudioJack4dpb-tokas_bp -> datum-rescue:AudioJack4dpb-tokas_bp
- U1, U2: symbol half-swept-rescue:ProMicro-kbd-bigblackpill-34key-rescue-sweepv2-rescue -> datum-rescue:ProMicro-kbd-bigblackpill-34key-rescue-sweepv2-rescue
Changed lines of the file:
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@@
     (pin "1")
   )
-  (symbol (lib_id "half-swept-rescue:ProMicro-kbd-bigblackpill-34key-rescue-sweepv2-rescue") (at 176.53 54.61 0) (unit 1)
+  (symbol (lib_id "datum-rescue:ProMicro-kbd-bigblackpill-34key-rescue-sweepv2-rescue") (at 176.53 54.61 0) (unit 1)
     (in_bom yes) (on_board yes)
     (property "Reference" "U1" (id 0) (at 176.53 25.5778 0)
@@
     (pin "3")
   )
-  (symbol (lib_id "half-swept-rescue:AudioJack4dpb-tokas_bp") (at 121.92 67.31 0) (unit 1)
+  (symbol (lib_id "datum-rescue:AudioJack4dpb-tokas_bp") (at 121.92 67.31 0) (unit 1)
     (in_bom yes) (on_board yes)
     (property "Reference" "J1" (id 0) (at 120.8278 59.055 0))
@@
     (pin "2")
   )
-  (symbol (lib_id "half-swept-rescue:ProMicro-kbd-bigblackpill-34key-rescue-sweepv2-rescue") (at 175.26 128.27 0) (unit 1)
+  (symbol (lib_id "datum-rescue:ProMicro-kbd-bigblackpill-34key-rescue-sweepv2-rescue") (at 175.26 128.27 0) (unit 1)
     (in_bom yes) (on_board yes)
     (property "Reference" "U2" (id 0) (at 175.26 99.2378 0)
@@
     (pin "2")
   )
-  (symbol (lib_id "half-swept-rescue:AudioJack4dpb-tokas_bp") (at 123.19 166.37 0) (unit 1)
+  (symbol (lib_id "datum-rescue:AudioJack4dpb-tokas_bp") (at 123.19 166.37 0) (unit 1)
     (in_bom yes) (on_board yes)
     (property "Reference" "J2" (id 0) (at 122.0978 158.115 0))
